Commit message: all macros are now modular

File: macros/depth_cam.xacro (robot description, xacro)
@@ -3,4 +3,5 @@
   <xacro:macro name="DepthCam" params="name
                link
+               optical_frame
                horizontal_fov
                img_width
@@ -17,6 +18,6 @@
                pointcloud_cuttoff">
   <gazebo reference="${link}">
-    <sensor type="DepthCam" name="${name}">
-        <always_on>true</always_on>
+    <sensor type="depth" name="${name}">
+        <always_on>1</always_on>
         <visualize>true</visualize>
         <camera>
@@ -38,5 +39,5 @@
                 <updateRate>${update_rate}</updateRate>
                 <cameraName>${name}</cameraName>
-                <frameName>camera_depth_optical_frame</frameName>
+                <frameName>${optical_frame}</frameName>
             <imageTopicName>${image_topic}</imageTopicName>
             <depthImageTopicName>${depth_topic}</depthImageTopicName>

File: macros/imu.xacro (robot description, xacro)
@@ -1,35 +1,35 @@
 <?xml version="1.0"?>
 <robot xmlns:xacro="http://www.ros.org/wiki/xacro" name="IMU" description="IMU sensor">
-	<xacro:macro name="imu" params="link hz topic">
- <gazebo reference="${link}">
-    <gravity>true</gravity>
-    <sensor name="imu_sensor" type="imu">
-      <always_on>true</always_on>
-      <update_rate>${hz}</update_rate>
-      <visualize>false</visualize>
-      <topic>IMU/data</topic>
-      <plugin filename="libgazebo_ros_imu_sensor.so" name="imu_plugin">
-        <topicName>${topic}</topicName>
-        <bodyName>${link}</bodyName>
-        <updateRateHZ>${hz}</updateRateHZ>
-        <gaussianNoise>0.01</gaussianNoise>
-        <xyzOffset>0 0 0</xyzOffset>
-        <rpyOffset>0 0 0</rpyOffset>
-        <frameName>${link}</frameName>
-      </plugin>
-      <pose>0 0 0 0 0 0</pose>
-    </sensor>
-  </gazebo>
-  <gazebo>
-        <plugin name="GazeboRosMagnetic" filename="libhector_gazebo_ros_magnetic.so">
-                <updateRate>50.0</updateRate>
-                <bodyName>${link}</bodyName>
-                <frameId>${link}</frameId>
-                <topicName>IMU/magnetic</topicName>
-                <offset>0 0 0</offset>
-                <drift>0.0 0.0 0.0</drift>
-                <gaussianNoise>1.3e-2 1.3e-2 1.3e-2</gaussianNoise>
+ <xacro:macro name="imu" params="link hz topic">
+    <gazebo reference="${link}">
+        <gravity>true</gravity>
+        <sensor name="imu_sensor" type="imu">
+        <always_on>true</always_on>
+        <update_rate>${hz}</update_rate>
+        <visualize>false</visualize>
+        <topic>${topic}/data</topic>
+        <plugin filename="libgazebo_ros_imu_sensor.so" name="imu_plugin">
+            <topicName>${topic}</topicName>
+            <bodyName>${link}</bodyName>
+            <updateRateHZ>${hz}</updateRateHZ>
+            <gaussianNoise>0.01</gaussianNoise>
+            <xyzOffset>0 0 0</xyzOffset>
+            <rpyOffset>0 0 0</rpyOffset>
+            <frameName>${link}</frameName>
         </plugin>
-</gazebo>
-	</xacro:macro>
+        <pose>0 0 0 0 0 0</pose>
+        </sensor>
+    </gazebo>
+    <gazebo>
+            <plugin name="GazeboRosMagnetic" filename="libhector_gazebo_ros_magnetic.so">
+                    <updateRate>50.0</updateRate>
+                    <bodyName>${link}</bodyName>
+                    <frameId>${link}</frameId>
+                    <topicName>${topic}/magnetic</topicName>
+                    <offset>0 0 0</offset>
+                    <drift>0.0 0.0 0.0</drift>
+                    <gaussianNoise>1.3e-2 1.3e-2 1.3e-2</gaussianNoise>
+            </plugin>
+    </gazebo>
+  </xacro:macro>
 </robot>

File: macros/lidar.xacro (robot description, xacro)
@@ -1,9 +1,10 @@
-<robot xmlns:xacro="http://www.ros.org/wiki/xacro" name="hokuyo" description="hokuyo">
-	<xacro:macro name="lidar" params="link topic samples resolution min_angle max_angle range_min range_max range_resolution">
+<?xml version="1.0"?>
+<robot xmlns:xacro="http://www.ros.org/wiki/xacro" name="lidar" description="LIDAR sensor">
+	<xacro:macro name="lidar" params="name link topic update_rate samples resolution min_angle max_angle range_min range_max range_resolution">
 		<gazebo reference="${link}">
-			<sensor type="ray" name="head_hokuyo_sensor">
+			<sensor type="ray" name="${name}">
 				<pose>0 0 0 0 0 0</pose>
 				<visualize>false</visualize>
-				<update_rate>10</update_rate>
+				<update_rate>${update_rate}</update_rate>
 				<ray>
 					<scan>

File: macros/urf.xacro (robot description, xacro)
@@ -1,9 +1,10 @@
-<robot xmlns:xacro="http://www.ros.org/wiki/xacro" name="URF" description="URF sensor">
- 	<xacro:macro name="urf" params=" name link topic fov min max">
+<?xml version="1.0"?>
+<robot xmlns:xacro="http://www.ros.org/wiki/xacro" name="urf_sensor" description="URF sensor">
+ 	<xacro:macro name="urf" params="name link topic fov min max update_rate">
 		<gazebo reference="${link}">
 			<material>Gazebo/Black</material>
 				<sensor type="ray" name="range">
 				<always_on>true</always_on>
-				<update_rate>10</update_rate>
+				<update_rate>${update_rate}</update_rate>
 				<pose>0 0 0 0 0 0</pose>
 				<visualize>false</visualize>
